File: PCB/SolasSense_Shamrock.kicad_pcb (KiCad board)
At the start: 2 copper layers, 86.7 x 75 mm, 15 parts, among them U1 ESP32-C3_SUPERMINI_TH

Commit message: Add files via upload
Connections:
- R11 pad 2: Net-(R11-Pad2) -> Net-(U1-GPIO2)
- R12 pad 1: Net-(R11-Pad2) -> Net-(U1-GPIO2)
- U1 pad 2: unconnected-(U1-GPIO2-Pad2) -> Net-(U1-GPIO2)
Routing:
- net Net-(U1-GPIO2): track 0.00 -> 65.0 mm, vias 0 -> 3
- net Net-(R11-Pad2): track 6.39 -> 0.00 mm
Changed lines of the file:
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@@
 			(outputformat 1)
 			(mirror no)
-			(drillshape 1)
+			(drillshape 0)
 			(scaleselection 1)
-			(outputdirectory "")
+			(outputdirectory "Shamrock-Gerber/")
 		)
 	)
@@
 	(net 21 "unconnected-(U1-GPIO10-Pad10)")
 	(net 22 "unconnected-(U1-GPIO20-Pad20)")
-	(net 23 "unconnected-(U1-GPIO2-Pad2)")
+	(net 23 "Net-(U1-GPIO2)")
 	(net 24 "unconnected-(U1-GPIO4-Pad4)")
 	(net 25 "unconnected-(U1-GPIO1-Pad1)")
-	(net 26 "Net-(R11-Pad2)")
 	(footprint "Resistor 220:RESC1005X35N"
 		(layer "F.Cu")
@@
 			(layers "*.Cu" "*.Mask")
 			(remove_unused_layers no)
-			(net 26 "Net-(R11-Pad2)")
+			(net 23 "Net-(U1-GPIO2)")
 			(pinfunction "1")
 			(pintype "unspecified")
@@
 			(layers "*.Cu" "*.Mask")
 			(remove_unused_layers no)
-			(net 23 "unconnected-(U1-GPIO2-Pad2)")
+			(net 23 "Net-(U1-GPIO2)")
 			(pinfunction "GPIO2")
 			(pintype "bidirectional")
@@
 			(size 0.51 0.6)
 			(layers "F.Cu" "F.Mask" "F.Paste")
-			(net 26 "Net-(R11-Pad2)")
+			(net 23 "Net-(U1-GPIO2)")
 			(pintype "passive")
 			(solder_mask_margin 0.102)
@@
 	)
 	(segment
-		(start 133.445 115.331826)
+		(start 132.681587 114.568413)
 		(end 129.573428 111.460254)
 		(width 0.2)
 		(layer "F.Cu")
-		(net 26)
+		(net 23)
+	)
+	(segment
+		(start 147.25 96.391915)
+		(end 150.420413 93.221502)
+		(width 0.2)
+		(layer "F.Cu")
+		(net 23)
+	)
+	(segment
+		(start 147.25 100)
+		(end 147.25 96.391915)
+		(width 0.2)
+		(layer "F.Cu")
+		(net 23)
+	)
+	(segment
+		(start 161.75 92.5)
+		(end 164.256661 89.993339)
+		(width 0.2)
+		(layer "F.Cu")
+		(net 23)
+	)
+	(segment
+		(start 132.681587 114.568413)
+		(end 147.25 100)
+		(width 0.2)
+		(layer "F.Cu")
+		(net 23)
+	)
+	(segment
+		(start 133.445 115.331826)
+		(end 132.681587 114.568413)
+		(width 0.2)
+		(layer "F.Cu")
+		(net 23)
+	)
+	(segment
+		(start 164.256661 89.993339)
+		(end 169.5 89.993339)
+		(width 0.2)
+		(layer "F.Cu")
+		(net 23)
 	)
 	(segment
@@
 		(width 0.2)
 		(layer "F.Cu")
-		(net 26)
+		(net 23)
+	)
+	(via
+		(at 169.5 89.993339)
+		(size 0.6)
+		(drill 0.3)
+		(layers "F.Cu" "B.Cu")
+		(net 23)
+	)
+	(via
+		(at 161.75 92.5)
+		(size 0.6)
+		(drill 0.3)
+		(layers "F.Cu" "B.Cu")
+		(net 23)
+	)
+	(via
+		(at 150.420413 93.221502)
+		(size 0.6)
+		(drill 0.3)
+		(layers "F.Cu" "B.Cu")
+		(net 23)
+	)
+	(segment
+		(start 169.5 90.833827)
+		(end 171.565784 92.899611)
+		(width 0.2)
+		(layer "B.Cu")
+		(net 23)
+	)
+	(segment
+		(start 150.420413 89.94915)
+		(end 152.487172 87.882391)
+		(width 0.2)
+		(layer "B.Cu")
+		(net 23)
+	)
+	(segment
+		(start 150.420413 93.221502)
+		(end 150.420413 89.94915)
+		(width 0.2)
+		(layer "B.Cu")
+		(net 23)
+	)
+	(segment
+		(start 157.132391 87.882391)
+		(end 161.75 92.5)
+		(width 0.2)
+		(layer "B.Cu")
+		(net 23)
+	)
+	(segment
+		(start 169.5 89.993339)
+		(end 169.5 90.833827)
+		(width 0.2)
+		(layer "B.Cu")
+		(net 23)
+	)
+	(segment
+		(start 152.487172 87.882391)
+		(end 157.132391 87.882391)
+		(width 0.2)
+		(layer "B.Cu")
+		(net 23)
 	)
 	(embedded_fonts no)

Commit message: Add files via upload
Parts:
- R1, R2, R3, R4, R5, R6, R7, R8, R9: footprint Resistor 220:RESC1005X35N -> Resistor_THT:R_Axial_DIN0204_L3.6mm_D1.6mm_P5.08mm_Vertical
- R11: footprint Resistor 10k:RESC1005X40N -> Resistor_THT:R_Axial_DIN0204_L3.6mm_D1.6mm_P5.08mm_Vertical
- moved R1 6.89 mm to (183.5, 80.0)
- moved R7 6.75 mm to (131.7, 96.0), turned to 180 degrees
- moved R6 6.25 mm to (151.2, 70.7), turned to 90 degrees
- moved R4 5.78 mm to (156.0, 69.7), turned to 90 degrees
- moved R9 5.24 mm to (131.5, 92.5), turned to 180 degrees
- moved R8 4.44 mm to (129.2, 86.8), turned to 180 degrees
- moved R3 4.31 mm to (147.2, 70.0), turned to 90 degrees
- moved R5 3.50 mm to (192.5, 91.0)
- moved R2 2.70 mm to (181.3, 83.8)
- moved R11 0.70 mm to (133.5, 116.8), turned to 180 degrees
Routing:
- net Net-(U1-GPIO6): track 118.2 -> 103.4 mm
- net Net-(U1-GPIO5): track 131.1 -> 117.1 mm
- net Net-(U1-GPIO7): track 114.8 -> 107.0 mm
- net Net-(D2-Pad2): track 6.69 -> 11.7 mm
- net GND: track 53.9 -> 50.5 mm
- net Net-(U1-GPIO2): track 65.0 -> 67.0 mm
- net Net-(D1-Pad2): track 4.82 -> 6.12 mm
- net Net-(D4-Pad1): track 4.58 -> 5.86 mm
- net Net-(D4-Pad4): track 4.99 -> 3.74 mm
- net Net-(D1-Pad1): track 7.46 -> 6.42 mm
- net Net-(D4-Pad2): track 5.77 -> 4.74 mm
- net Net-(D2-Pad1): track 5.64 -> 6.59 mm
- net Net-(D2-Pad4): track 7.05 -> 7.94 mm
- net Net-(D1-Pad4): track 4.35 -> 5.11 mm
