File: PCB/SolasSense_Shamrock.kicad_sch (KiCad schematic)
At the start: 15 parts, among them U1 ESP32-C3_SUPERMINI_TH

Commit message: Add files via upload
Connections:
- net at R11.2, R12.1: now also U1.2 (GPIO2)
Changed lines of the file:
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@@
 	(paper "A4")
 	(junction
+		(at 82.55 73.66)
+		(diameter 0)
+		(color 0 0 0 0)
+	)
+	(junction
 		(at 142.24 91.44)
 		(diameter 0)
@@
 	(wire
 		(pts
+			(xy 90.17 73.66) (xy 90.17 54.61)
+		)
+		(stroke
+			(width 0)
+			(type default)
+		)
+	)
+	(wire
+		(pts
 			(xy 153.67 83.82) (xy 153.67 96.52)
 		)
@@
 	(wire
 		(pts
+			(xy 82.55 73.66) (xy 90.17 73.66)
+		)
+		(stroke
+			(width 0)
+			(type default)
+		)
+	)
+	(wire
+		(pts
 			(xy 95.25 96.52) (xy 95.25 62.23)
 		)
@@
 	(wire
 		(pts
+			(xy 90.17 54.61) (xy 102.87 54.61)
+		)
+		(stroke
+			(width 0)
+			(type default)
+		)
+	)
+	(wire
+		(pts
 			(xy 184.15 80.01) (xy 184.15 83.82)
 		)
@@
 	(wire
 		(pts
+			(xy 82.55 73.66) (xy 82.55 74.93)
+		)
+		(stroke
+			(width 0)
+			(type default)
+		)
+	)
+	(wire
+		(pts
 			(xy 99.06 91.44) (xy 99.06 64.77)
 		)
@@
 	(wire
 		(pts
-			(xy 82.55 71.12) (xy 82.55 74.93)
-		)
-		(stroke
+			(xy 82.55 71.12) (xy 82.55 73.66)
+		)
+		(stroke

Commit message: Add files via upload
Parts:
- R1, R2, R3, R4, R5, R6, R7, R8, R9: footprint Resistor 220:RESC1005X35N -> Resistor_THT:R_Axial_DIN0204_L3.6mm_D1.6mm_P5.08mm_Vertical
- R11: footprint Resistor 10k:RESC1005X40N -> Resistor_THT:R_Axial_DIN0204_L3.6mm_D1.6mm_P5.08mm_Vertical
Changed lines of the file:
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@@
 			)
 		)
-		(property "Footprint" "Resistor 220:RESC1005X35N"
+		(property "Footprint" "Resistor_THT:R_Axial_DIN0204_L3.6mm_D1.6mm_P5.08mm_Vertical"
 			(at 173.99 105.41 0)
 			(effects
@@
 			)
 		)
-		(property "Footprint" "Resistor 220:RESC1005X35N"
+		(property "Footprint" "Resistor_THT:R_Axial_DIN0204_L3.6mm_D1.6mm_P5.08mm_Vertical"
 			(at 175.26 39.37 0)
 			(effects
@@
 			)
 		)
-		(property "Footprint" "Resistor 220:RESC1005X35N"
+		(property "Footprint" "Resistor_THT:R_Axial_DIN0204_L3.6mm_D1.6mm_P5.08mm_Vertical"
 			(at 175.26 72.39 0)
 			(effects
@@
 			)
 		)
-		(property "Footprint" "Resistor 220:RESC1005X35N"
+		(property "Footprint" "Resistor_THT:R_Axial_DIN0204_L3.6mm_D1.6mm_P5.08mm_Vertical"
 			(at 173.99 95.25 0)
 			(effects
@@
 			)
 		)
-		(property "Footprint" "Resistor 10k:RESC1005X40N"
+		(property "Footprint" "Resistor_THT:R_Axial_DIN0204_L3.6mm_D1.6mm_P5.08mm_Vertical"
 			(at 82.55 85.09 0)
 			(effects
@@
 			)
 		)
-		(property "Footprint" "Resistor 220:RESC1005X35N"
+		(property "Footprint" "Resistor_THT:R_Axial_DIN0204_L3.6mm_D1.6mm_P5.08mm_Vertical"
 			(at 173.99 83.82 0)
 			(effects
@@
 			)
 		)
-		(property "Footprint" "Resistor 220:RESC1005X35N"
+		(property "Footprint" "Resistor_THT:R_Axial_DIN0204_L3.6mm_D1.6mm_P5.08mm_Vertical"
 			(at 175.26 29.21 0)
 			(effects
@@
 			)
 		)
-		(property "Footprint" "Resistor 220:RESC1005X35N"
+		(property "Footprint" "Resistor_THT:R_Axial_DIN0204_L3.6mm_D1.6mm_P5.08mm_Vertical"
 			(at 172.72 116.84 0)
 			(effects
@@
 			)
 		)
-		(property "Footprint" "Resistor 220:RESC1005X35N"
+		(property "Footprint" "Resistor_THT:R_Axial_DIN0204_L3.6mm_D1.6mm_P5.08mm_Vertical"
 			(at 175.26 62.23 0)
 			(effects
@@
 			)
 		)
-		(property "Footprint" "Resistor 220:RESC1005X35N"
+		(property "Footprint" "Resistor_THT:R_Axial_DIN0204_L3.6mm_D1.6mm_P5.08mm_Vertical"
 			(at 173.99 50.8 0)
 			(effects
